File: unkeyable/RP2040_minimal.kicad_sch (KiCad schematic)
At the start: 23 parts, among them U2 W25Q128JVS, U3 RP2040, Y1 ABM8-272-T3

Commit message: layout
Parts:
- removed C1, C2: 15p, Capacitor_SMD:C_0402_1005Metric, symbol Device:C
- removed C10, C8: 1u, Capacitor_SMD:C_0402_1005Metric, symbol Device:C
- removed C11, C12, C13, C14, C15, C16, C5, C6, C7, C9: 100n, Capacitor_SMD:C_0402_1005Metric, symbol Device:C
- removed JP1: Jumper_2_Small_Open, symbol Jumper:Jumper_2_Small_Open
- removed R1, R3: 1k, Resistor_SMD:R_0402_1005Metric, symbol Device:R
- removed R2: DNF, Resistor_SMD:R_0402_1005Metric, symbol Device:R
- removed R4, R5: 27, Resistor_SMD:R_0402_1005Metric, symbol Device:R
- removed U2: W25Q128JVS, Package_SO:SOIC-8_5.23x5.23mm_P1.27mm, symbol Memory_Flash:W25Q128JVS
- removed U3: RP2040, RP2040_minimal:RP2040-QFN-56, symbol MCU_RaspberryPi_RP2040:RP2040
- removed Y1: ABM8-272-T3, Crystal:Crystal_SMD_3225-4Pin_3.2x2.5mm, symbol Device:Crystal_GND24
- added J1, J2: Conn_01x13, Connector_PinSocket_2.54mm:PinSocket_1x13_P2.54mm_Vertical, symbol Connector_Generic:Conn_01x13
Connections:
- net +3V3: now also J2.5 (Pin_5)
- net GND: now also J1.4 (Pin_4), J1.5 (Pin_5), J2.3 (Pin_3)
- net GPIO0: now also J1.2 (Pin_2)
- net GPIO1: now also J1.3 (Pin_3)
- net GPIO10: now also J2.13 (Pin_13)
- net GPIO18: now also J2.10 (Pin_10)
- net GPIO19: now also J2.12 (Pin_12)
- net GPIO2: now also J1.6 (Pin_6)
- net GPIO20: now also J2.11 (Pin_11)
- net GPIO26_ADC0: now also J2.9 (Pin_9)
- net GPIO27_ADC1: now also J2.8 (Pin_8)
- net GPIO28_ADC2: now also J2.7 (Pin_7)
- net GPIO29_ADC3: now also J2.6 (Pin_6)
- net GPIO3: now also J1.7 (Pin_7)
- net GPIO4: now also J1.8 (Pin_8)
- net GPIO5: now also J1.9 (Pin_9)
- net GPIO6: now also J1.10 (Pin_10)
- net GPIO7: now also J1.11 (Pin_11)
- net GPIO8: now also J1.12 (Pin_12)
- net GPIO9: now also J1.13 (Pin_13)
- net USB_D+: now also J1.1 (Pin_1)
- net USB_D-: now also J2.1 (Pin_1)
- new net +5V: J2.2 (Pin_2)
- new net RESET: J2.4 (Pin_4)
Other:
- note removed: "Crystal"
- note removed: "Flash"
- note removed: "Make sure C10 is close to pin 44 of RP2040"
- note removed: "Make sure C8 is close to pin 45 of RP2040"
- note removed: "Make sure R3 and R4 are close to RP2040"
