File: unkeyable/Switch_Matrix.kicad_sch (KiCad schematic)
At the start: 48 parts, among them SW1 1, SW10 F, SW11 J, SW12 K, SW2 C, SW3 3, SW4 Q, SW5 W, SW6 E, SW7 A, SW8 S, SW9 D

Commit message: layout
Parts:
- removed C19, C20, C21, C22, C23, C24, C25, C26, C27, C28, C3, C4: 0.1uF, symbol Device:C_Small
- removed D13, D14, D15, D16, D17, D18, D19, D20, D21, D22, D23, D24: WS2812B-2020, LED_SMD:LED_WS2812B_PLCC4_5.0x5.0mm_P3.2mm, symbol LED:WS2812B-2020
- added D11, D12, D17, D5, D6: 1n4148, Diode_SMD:D_SOD-323, symbol Device:D
- added SW11: S, Button_Switch_Keyboard:SW_Cherry_MX_1.00u_PCB, symbol Switch:SW_Push
- added SW12: D, Button_Switch_Keyboard:SW_Cherry_MX_1.00u_PCB, symbol Switch:SW_Push
- added SW17: SPACE, Button_Switch_Keyboard:SW_Cherry_MX_6.25u_PCB, symbol Switch:SW_Push
- added SW5: SHIFT, Button_Switch_Keyboard:SW_Cherry_MX_1.75u_PCB, symbol Switch:SW_Push
- added SW6: Q, Button_Switch_Keyboard:SW_Cherry_MX_1.00u_PCB, symbol Switch:SW_Push
- D1, D2, D3, D4: value D -> 1n4148; footprint (none) -> Diode_SMD:D_SOD-323
- D10: renamed from D8; value D -> 1n4148; footprint (none) -> Diode_SMD:D_SOD-323
- D13: renamed from D9; value D -> 1n4148; footprint (none) -> Diode_SMD:D_SOD-323
- D14: renamed from D10; value D -> 1n4148; footprint (none) -> Diode_SMD:D_SOD-323
- D15: renamed from D11; value D -> 1n4148; footprint (none) -> Diode_SMD:D_SOD-323
- D16: renamed from D12; value D -> 1n4148; footprint (none) -> Diode_SMD:D_SOD-323
- D7: renamed from D5; value D -> 1n4148; footprint (none) -> Diode_SMD:D_SOD-323
- D8: renamed from D6; value D -> 1n4148; footprint (none) -> Diode_SMD:D_SOD-323
- D9: renamed from D7; value D -> 1n4148; footprint (none) -> Diode_SMD:D_SOD-323
- SW1: value 1 -> ESC; footprint Button_Switch_Keyboard:SW_Cherry_MX_1.00u_PCB -> Button_Switch_Keyboard:SW_Cherry_MX_1.75u_PCB
- SW10: renamed from SW8; value S -> A
- SW13: renamed from SW9; value D -> F
- SW14: renamed from SW10; value F -> J
- SW15: renamed from SW11; value J -> K
- SW16: renamed from SW12; value K -> ALT; footprint Button_Switch_Keyboard:SW_Cherry_MX_1.00u_PCB -> Button_Switch_Keyboard:SW_Cherry_MX_1.75u_PCB
- SW2: value C -> 1
- SW3: value 3 -> C
- SW4: value Q -> 3
- SW9: renamed from SW7; value A -> CTRL; footprint Button_Switch_Keyboard:SW_Cherry_MX_1.00u_PCB -> Button_Switch_Keyboard:SW_Cherry_MX_1.75u_PCB
- renumbered SW5 to SW7, SW6 to SW8
Connections:
- net COL_1: now also SW5.1; no longer SW14.1, SW4.1
- net COL_2: now also SW6.1; no longer SW15.1, SW7.1
- net COL_3: now also SW7.1, SW11.1; no longer SW13.1, SW16.1, SW8.1
- net ROW_1: now also D13.1 (K), D16.1 (K), D4.1 (K)
- net ROW_2: now also D14.1 (K), D17.1 (K), D5.1 (K), D6.1 (K); no longer D4.1 (K)
- net ROW_3: now also D15.1 (K), D11.1 (K), D12.1 (K); no longer D13.1 (K)
- removed net ROW_4: D14.1 (K), D15.1 (K), D16.1 (K)
- new net: D11.2 (A), SW11.2
- new net: D5.2 (A), SW5.2
- new net: D17.2 (A), SW17.2
- new net: D6.2 (A), SW6.2
- new net: D12.2 (A), SW12.2
- new net COL_4: SW12.1, SW4.1, SW8.1
- new net COL_5: SW13.1, SW14.1, SW15.1
- new net COL_6: SW16.1, SW17.1
- no-connect marks 1 -> 0
Other:
- moved on the sheet: D10, D13, D14, D15, D16, D3, D4, D7, D8, D9, SW10, SW13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
