File: unkeyable/unkeyable.kicad_pcb (KiCad board)
At the start: 2 copper layers, 0 parts

Commit message: layout
Parts:
- added D1: 1n4148, Diode_SMD:D_SOD-323, B.Cu at (64.5, 51.2)
- added D10: 1n4148, Diode_SMD:D_SOD-323, B.Cu at (90.7, 89.3)
- added D11: 1n4148, Diode_SMD:D_SOD-323, B.Cu at (109.8, 89.3)
- added D12: 1n4148, Diode_SMD:D_SOD-323, B.Cu at (128.8, 89.3)
- added D13: 1n4148, Diode_SMD:D_SOD-323, B.Cu at (147.9, 89.3)
- added D14: 1n4148, Diode_SMD:D_SOD-323, B.Cu at (205.0, 89.3)
- added D15: 1n4148, Diode_SMD:D_SOD-323, B.Cu at (224.1, 89.3)
- added D16: 1n4148, Diode_SMD:D_SOD-323, B.Cu at (64.5, 108.3)
- added D17: 1n4148, Diode_SMD:D_SOD-323, B.Cu at (178.8, 108.3)
- added D2: 1n4148, Diode_SMD:D_SOD-323, B.Cu at (90.7, 51.2)
- added D3: 1n4148, Diode_SMD:D_SOD-323, B.Cu at (109.8, 51.2)
- added D4: 1n4148, Diode_SMD:D_SOD-323, B.Cu at (128.8, 51.2)
- added D5: 1n4148, Diode_SMD:D_SOD-323, B.Cu at (64.5, 70.2)
- added D6: 1n4148, Diode_SMD:D_SOD-323, B.Cu at (90.7, 70.2)
- added D7: 1n4148, Diode_SMD:D_SOD-323, B.Cu at (109.8, 70.2)
- added D8: 1n4148, Diode_SMD:D_SOD-323, B.Cu at (128.8, 70.2)
- added D9: 1n4148, Diode_SMD:D_SOD-323, B.Cu at (64.5, 89.3)
- added J1: Conn_01x13, Connector_PinSocket_2.54mm:PinSocket_1x13_P2.54mm_Vertical, B.Cu at (150.8, 46.7)
- added J2: Conn_01x13, Connector_PinSocket_2.54mm:PinSocket_1x13_P2.54mm_Vertical, B.Cu at (135.6, 46.7)
- added REF**: MountingHole_2.2mm_M2, MountingHole:MountingHole_2.2mm_M2, F.Cu at (193.2, 118.2)
- added REF**: MountingHole_2.2mm_M2, MountingHole:MountingHole_2.2mm_M2, F.Cu at (228.5, 99.9)
- added REF**: MountingHole_2.2mm_M2, MountingHole:MountingHole_2.2mm_M2, F.Cu at (93.2, 118.2)
- added REF**: MountingHole_2.2mm_M2, MountingHole:MountingHole_2.2mm_M2, F.Cu at (228.5, 80.8)
- added REF**: MountingHole_2.2mm_M2, MountingHole:MountingHole_2.2mm_M2, F.Cu at (142.8, 118.2)
- added REF**: MountingHole_2.2mm_M2, MountingHole:MountingHole_2.2mm_M2, F.Cu at (228.5, 61.9)
- added REF**: MountingHole_2.2mm_M2, MountingHole:MountingHole_2.2mm_M2, F.Cu at (178.3, 80.9)
- added REF**: MountingHole_2.2mm_M2, MountingHole:MountingHole_2.2mm_M2, F.Cu at (42.5, 118.2)
- added REF**: MountingHole_2.2mm_M2, MountingHole:MountingHole_2.2mm_M2, F.Cu at (42.5, 45.2)
- added REF**: MountingHole_2.2mm_M2, MountingHole:MountingHole_2.2mm_M2, F.Cu at (42.5, 80.8)
- added REF**: MountingHole_2.2mm_M2, MountingHole:MountingHole_2.2mm_M2, F.Cu at (193.6, 45.2)
- added REF**: MountingHole_2.2mm_M2, MountingHole:MountingHole_2.2mm_M2, F.Cu at (228.5, 118.2)
- added REF**: MountingHole_2.2mm_M2, MountingHole:MountingHole_2.2mm_M2, F.Cu at (42.5, 61.8)
- added REF**: MountingHole_2.2mm_M2, MountingHole:MountingHole_2.2mm_M2, F.Cu at (228.5, 45.2)
- added REF**: MountingHole_2.2mm_M2, MountingHole:MountingHole_2.2mm_M2, F.Cu at (142.8, 45.2)
- added REF**: MountingHole_2.2mm_M2, MountingHole:MountingHole_2.2mm_M2, F.Cu at (42.5, 99.9)
- added REF**: MountingHole_2.2mm_M2, MountingHole:MountingHole_2.2mm_M2, F.Cu at (92.6, 80.9)
- added SW1: ESC, Button_Switch_Keyboard:SW_Cherry_MX_1.75u_PCB, F.Cu at (59.4, 47.2)
- added SW10: A, Button_Switch_Keyboard:SW_Cherry_MX_1.00u_PCB, F.Cu at (85.6, 85.3)
- added SW11: S, Button_Switch_Keyboard:SW_Cherry_MX_1.00u_PCB, F.Cu at (104.7, 85.3)
- added SW12: D, Button_Switch_Keyboard:SW_Cherry_MX_1.00u_PCB, F.Cu at (123.7, 85.3)
- added SW13: F, Button_Switch_Keyboard:SW_Cherry_MX_1.00u_PCB, F.Cu at (142.8, 85.3)
- added SW14: J, Button_Switch_Keyboard:SW_Cherry_MX_1.00u_PCB, F.Cu at (199.9, 85.3)
- added SW15: K, Button_Switch_Keyboard:SW_Cherry_MX_1.00u_PCB, F.Cu at (219.0, 85.3)
- added SW16: ALT, Button_Switch_Keyboard:SW_Cherry_MX_1.75u_PCB, F.Cu at (59.4, 104.3)
- added SW17: SPACE, Button_Switch_Keyboard:SW_Cherry_MX_6.25u_PCB, F.Cu at (173.7, 104.3)
- added SW2: 1, Button_Switch_Keyboard:SW_Cherry_MX_1.00u_PCB, F.Cu at (85.6, 47.2)
- added SW3: C, Button_Switch_Keyboard:SW_Cherry_MX_1.00u_PCB, F.Cu at (104.7, 47.2)
- added SW4: 3, Button_Switch_Keyboard:SW_Cherry_MX_1.00u_PCB, F.Cu at (123.7, 47.2)
- added SW5: SHIFT, Button_Switch_Keyboard:SW_Cherry_MX_1.75u_PCB, F.Cu at (59.4, 66.2)
- added SW6: Q, Button_Switch_Keyboard:SW_Cherry_MX_1.00u_PCB, F.Cu at (85.6, 66.2)
- added SW7: W, Button_Switch_Keyboard:SW_Cherry_MX_1.00u_PCB, F.Cu at (104.7, 66.2)
- added SW8: E, Button_Switch_Keyboard:SW_Cherry_MX_1.00u_PCB, F.Cu at (123.7, 66.2)
- added SW9: CTRL, Button_Switch_Keyboard:SW_Cherry_MX_1.75u_PCB, F.Cu at (59.4, 85.3)
Routing:
- net /RP2040/GPIO7: track 0.00 -> 227.6 mm, vias 0 -> 1
- net /RP2040/GPIO8: track 0.00 -> 213.8 mm, vias 0 -> 1
- net /RP2040/GPIO9: track 0.00 -> 190.4 mm
- net /RP2040/GPIO5: track 0.00 -> 162.2 mm, vias 0 -> 1
- net /RP2040/GPIO29_ADC3: track 0.00 -> 130.4 mm
- net /RP2040/GPIO28_ADC2: track 0.00 -> 105.4 mm
- net /RP2040/GPIO4: track 0.00 -> 100.3 mm
- net /RP2040/GPIO27_ADC1: track 0.00 -> 87.2 mm
- net /RP2040/GPIO26_ADC0: track 0.00 -> 50.3 mm
- net GND: track 0.00 -> 18.8 mm
- net Net-(D7-A): track 0.00 -> 11.6 mm
- net Net-(D17-A): track 0.00 -> 11.6 mm
- net Net-(D15-A): track 0.00 -> 11.6 mm
- net Net-(D13-A): track 0.00 -> 11.6 mm
- net Net-(D11-A): track 0.00 -> 11.6 mm
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Other:
- board outline added: 191 x 78 mm

Commit message: fabrication output file
Parts:
- removed the REF** at (193.2, 118.2)
- removed the REF** at (93.2, 118.2)
- removed the REF** at (228.5, 61.9)
- removed the REF** at (193.6, 45.2)
- removed the REF** at (42.5, 61.8)
- added REF**: Fiducial_0.5mm_Mask1.5mm, Fiducial:Fiducial_0.5mm_Mask1.5mm, B.Cu at (179.3, 62.9)
- moved REF** 11.3 mm to (42.5, 69.5)
- moved REF** 11.3 mm to (228.5, 69.5)
- moved REF** 6.03 mm to (42.5, 93.9)
- moved REF** 6.03 mm to (228.5, 93.9)
- moved REF** 0.10 mm to (178.4, 80.9)
Routing:
- net /RP2040/GPIO8: track 213.8 -> 211.2 mm
- net /RP2040/GPIO7: track 227.6 -> 226.0 mm
- net /RP2040/GPIO9: track 190.4 -> 188.8 mm
- net /RP2040/GPIO29_ADC3: track 130.4 -> 129.7 mm
- net /RP2040/GPIO27_ADC1: track 87.2 -> 86.5 mm
- net /RP2040/GPIO5: track 162.2 -> 161.5 mm
- net /RP2040/GPIO28_ADC2: track 105.4 -> 104.9 mm
